File: nixie/200VDCDC/200VDCDC.sch (KiCad schematic (older format))
At the start: 20 parts, among them J1 +12V, J2 +200V, Q1 2SA1015, Q2 TK10A60D, U1 NJM2360

Commit message: 2020/03/31 DC/DC SMD
Parts:
- C1: footprint (none) -> Capacitor_SMD:CP_Elec_10x12.5
- C2, C3, C4: footprint (none) -> Capacitor_SMD:C_0603_1608Metric_Pad1.05x0.95mm_HandSolder
- C5: footprint (none) -> Capacitor_THT:CP_Radial_D18.0mm_P7.50mm
- D1: footprint Diode_SMD:D_SOD-123 -> Diode_THT:D_A-405_P7.62mm_Horizontal
- D2: footprint Diode_SMD:D_SOD-123 -> Diode_THT:D_T-1_P10.16mm_Horizontal
- J1, J2: footprint (none) -> Connector_PinHeader_2.54mm:PinHeader_1x02_P2.54mm_Vertical
- L1: footprint (none) -> Inductor_SMD:L_12x12mm_H8mm
- Q1: footprint (none) -> Package_TO_SOT_THT:TO-92_Inline_Wide
- Q2: footprint (none) -> Package_TO_SOT_THT:TO-3PB-3_Vertical
- R1, R2, R3, R4, R5, R6: footprint (none) -> Resistor_SMD:R_0603_1608Metric_Pad1.05x0.95mm_HandSolder
- RV1: footprint (none) -> Potentiometer_THT:Potentiometer_ACP_CA6-H2,5_Horizontal
- U1: footprint (none) -> Package_DIP:DIP-8_W8.89mm_SMDSocket_LongPads
Changed lines of the file:
@@
 EESchema Schematic File Version 4
-EELAYER 29 0
+EELAYER 30 0
 EELAYER END
 $Descr A4 11693 8268
@@
 F 0 "U1" H 4550 4365 50  0000 C CNN
 F 1 "NJM2360" H 4550 4274 50  0000 C CNN
-F 2 "" H 4550 3650 50  0001 C CNN
+F 2 "Package_DIP:DIP-8_W8.89mm_SMDSocket_LongPads" H 4550 3650 50  0001 C CNN
 F 3 "" H 4550 3650 50  0001 C CNN
 	1    4550 3800
@@
 F 0 "L1" V 6190 2850 50  0000 C CNN
 F 1 "470u" V 6099 2850 50  0000 C CNN
-F 2 "" H 6000 2850 50  0001 C CNN
-F 3 "~" H 6000 2850 50  0001 C CNN
+F 2 "Inductor_SMD:L_12x12mm_H8mm" H 6000 2850 50  0001 C CNN
+F 3 "http://akizukidenshi.com/catalog/g/gP-13969/" H 6000 2850 50  0001 C CNN
 	1    6000 2850
 	0    -1   -1   0
@@
 F 0 "R3" H 5470 3246 50  0000 L CNN
 F 1 "680" H 5470 3155 50  0000 L CNN
-F 2 "" V 5330 3200 50  0001 C CNN
+F 2 "Resistor_SMD:R_0603_1608Metric_Pad1.05x0.95mm_HandSolder" V 5330 3200 50  0001 C CNN
 F 3 "~" H 5400 3200 50  0001 C CNN
 	1    5400 3200
@@
 F 0 "R2" H 3770 3246 50  0000 L CNN
 F 1 "1k" H 3770 3155 50  0000 L CNN
-F 2 "" V 3630 3200 50  0001 C CNN
+F 2 "Resistor_SMD:R_0603_1608Metric_Pad1.05x0.95mm_HandSolder" V 3630 3200 50  0001 C CNN
 F 3 "~" H 3700 3200 50  0001 C CNN
 	1    3700 3200
@@
 F 0 "Q1" H 6791 4504 50  0000 L CNN
 F 1 "2SA1015" H 6791 4595 50  0000 L CNN
-F 2 "" H 6800 4650 50  0001 C CNN
+F 2 "Package_TO_SOT_THT:TO-92_Inline_Wide" H 6800 4650 50  0001 C CNN
 F 3 "~" H 6600 4550 50  0001 C CNN
 	1    6600 4550
@@
 F 0 "D1" V 6104 4280 50  0000 L CNN
 F 1 "1N4148" V 6195 4280 50  0000 L CNN
-F 2 "Diode_SMD:D_SOD-123" H 6150 4025 50  0001 C CNN
-F 3 "https://www.vishay.com/docs/85748/1n4148w.pdf" H 6150 4200 50  0001 C CNN
+F 2 "Diode_THT:D_A-405_P7.62mm_Horizontal" H 6150 4025 50  0001 C CNN
+F 3 "http://akizukidenshi.com/catalog/g/gI-00941/" H 6150 4200 50  0001 C CNN
 	1    6150 4200
 	0    1    1    0
@@
 F 0 "R4" H 6220 4896 50  0000 L CNN
 F 1 "1k" H 6220 4805 50  0000 L CNN
-F 2 "" V 6080 4850 50  0001 C CNN
+F 2 "Resistor_SMD:R_0603_1608Metric_Pad1.05x0.95mm_HandSolder" V 6080 4850 50  0001 C CNN
 F 3 "~" H 6150 4850 50  0001 C CNN
 	1    6150 4850
@@
 F 0 "Q2" H 7556 3696 50  0000 L CNN
 F 1 "TK10A60D" H 7556 3605 50  0000 L CNN
-F 2 "" H 7550 3750 50  0001 C CNN
-F 3 "~" H 7350 3650 50  0001 C CNN
+F 2 "Package_TO_SOT_THT:TO-3PB-3_Vertical" H 7550 3750 50  0001 C CNN
+F 3 "http://akizukidenshi.com/catalog/g/gI-08418/" H 7350 3650 50  0001 C CNN
 	1    7350 3650
 	1    0    0    -1
@@
 F 0 "D2" H 7900 2633 50  0000 C CNN
 F 1 "UF2010" H 7900 2724 50  0000 C CNN
-F 2 "Diode_SMD:D_SOD-123" H 7900 2675 50  0001 C CNN
-F 3 "https://www.vishay.com/docs/85748/1n4148w.pdf" H 7900 2850 50  0001 C CNN
+F 2 "Diode_THT:D_T-1_P10.16mm_Horizontal" H 7900 2675 50  0001 C CNN
+F 3 "http://akizukidenshi.com/catalog/g/gI-00124/" H 7900 2850 50  0001 C CNN
 	1    7900 2850
 	-1   0    0    1
@@
 F 0 "R5" H 8570 3396 50  0000 L CNN
 F 1 "470k" H 8570 3305 50  0000 L CNN
-F 2 "" V 8430 3350 50  0001 C CNN
+F 2 "Resistor_SMD:R_0603_1608Metric_Pad1.05x0.95mm_HandSolder" V 8430 3350 50  0001 C CNN
 F 3 "~" H 8500 3350 50  0001 C CNN
 	1    8500 3350
@@
 F 0 "R6" H 8570 4896 50  0000 L CNN
 F 1 "2.2k" H 8570 4805 50  0000 L CNN
-F 2 "" V 8430 4850 50  0001 C CNN
+F 2 "Resistor_SMD:R_0603_1608Metric_Pad1.05x0.95mm_HandSolder" V 8430 4850 50  0001 C CNN
 F 3 "~" H 8500 4850 50  0001 C CNN
 	1    8500 4850
@@
 F 0 "RV1" H 8430 4054 50  0000 R CNN
 F 1 "50k" H 8430 4145 50  0000 R CNN
-F 2 "" H 8500 4100 50  0001 C CNN
-F 3 "~" H 8500 4100 50  0001 C CNN
+F 2 "Potentiometer_THT:Potentiometer_ACP_CA6-H2,5_Horizontal" H 8500 4100 50  0001 C CNN
+F 3 "http://akizukidenshi.com/catalog/g/gP-03281/" H 8500 4100 50  0001 C CNN
 	1    8500 4100
 	-1   0    0    1
@@
 F 0 "R1" V 2643 5400 50  0000 C CNN
 F 1 "0" V 2734 5400 50  0000 C CNN
-F 2 "" V 2780 5400 50  0001 C CNN
+F 2 "Resistor_SMD:R_0603_1608Metric_Pad1.05x0.95mm_HandSolder" V 2780 5400 50  0001 C CNN
 F 3 "~" H 2850 5400 50  0001 C CNN
 	1    2850 5400
@@
 F 0 "C1" H 2015 4896 50  0000 L CNN
 F 1 "100u" H 2015 4805 50  0000 L CNN
-F 2 "" H 1900 4850 50  0001 C CNN
-F 3 "~" H 1900 4850 50  0001 C CNN
+F 2 "Capacitor_SMD:CP_Elec_10x12.5" H 1900 4850 50  0001 C CNN
+F 3 "http://akizukidenshi.com/catalog/g/gP-12940/" H 1900 4850 50  0001 C CNN
 	1    1900 4850
 	1    0    0    -1
@@
 F 0 "J1" H 1018 4417 50  0000 C CNN
 F 1 "+12V" H 1018 4326 50  0000 C CNN
-F 2 "" H 1100 4200 50  0001 C CNN
+F 2 "Connector_PinHeader_2.54mm:PinHeader_1x02_P2.54mm_Vertical" H 1100 4200 50  0001 C CNN
 F 3 "~" H 1100 4200 50  0001 C CNN
 	1    1100 4200
@@
 F 0 "J2" H 9780 4092 50  0000 L CNN
 F 1 "+200V" H 9780 4001 50  0000 L CNN
-F 2 "" H 9700 4100 50  0001 C CNN
+F 2 "Connector_PinHeader_2.54mm:PinHeader_1x02_P2.54mm_Vertical" H 9700 4100 50  0001 C CNN
 F 3 "~" H 9700 4100 50  0001 C CNN
 	1    9700 4100
@@
 F 0 "C2" H 2515 4896 50  0000 L CNN
 F 1 "100n" H 2515 4805 50  0000 L CNN
-F 2 "" H 2438 4700 50  0001 C CNN
-F 3 "~" H 2400 4850 50  0001 C CNN
+F 2 "Capacitor_SMD:C_0603_1608Metric_Pad1.05x0.95mm_HandSolder" H 2438 4700 50  0001 C CNN
+F 3 "http://akizukidenshi.com/catalog/g/gP-13374/" H 2400 4850 50  0001 C CNN
 	1    2400 4850
 	1    0    0    -1
@@
 F 0 "C3" H 3365 4896 50  0000 L CNN
 F 1 "680p" H 3365 4805 50  0000 L CNN
-F 2 "" H 3288 4700 50  0001 C CNN
-F 3 "~" H 3250 4850 50  0001 C CNN
+F 2 "Capacitor_SMD:C_0603_1608Metric_Pad1.05x0.95mm_HandSolder" H 3288 4700 50  0001 C CNN
+F 3 "http://akizukidenshi.com/catalog/g/gP-05588/" H 3250 4850 50  0001 C CNN
 	1    3250 4850
 	1    0    0    -1
@@
 F 0 "C5" H 9065 4196 50  0000 L CNN
 F 1 "100u" H 9065 4105 50  0000 L CNN
-F 2 "" H 8950 4150 50  0001 C CNN
-F 3 "~" H 8950 4150 50  0001 C CNN
+F 2 "Capacitor_THT:CP_Radial_D18.0mm_P7.50mm" H 8950 4150 50  0001 C CNN
+F 3 "http://akizukidenshi.com/catalog/g/gP-10604/" H 8950 4150 50  0001 C CNN
 	1    8950 4150
 	1    0    0    -1
@@
 F 0 "C4" H 5465 4846 50  0000 L CNN
 F 1 "100n" H 5465 4755 50  0000 L CNN
-F 2 "" H 5388 4650 50  0001 C CNN
-F 3 "~" H 5350 4800 50  0001 C CNN
+F 2 "Capacitor_SMD:C_0603_1608Metric_Pad1.05x0.95mm_HandSolder" H 5388 4650 50  0001 C CNN
+F 3 "http://akizukidenshi.com/catalog/g/gP-13377/" H 5350 4800 50  0001 C CNN
 	1    5350 4800
 	1    0    0    -1
